File: Simple_Curve_Tracer/Simple_Curve_Tracer.kicad_sch (KiCad schematic)
At the start: 25 parts, among them Q1 PN2222A, Q2 2N3905, Q3 2N3905, Q4 PN2222A, U1 LM358, U2 74LS393

Commit message: various additions
Parts:
- added C2: 10nF (103), Capacitor_THT:C_Rect_L7.0mm_W3.5mm_P5.00mm, symbol Device:C_Small
- added C3: 100nF (104), Capacitor_THT:C_Rect_L7.0mm_W3.5mm_P5.00mm, symbol Device:C_Small
- added J1: DUT, Connector_PinSocket_2.54mm:PinSocket_1x05_P2.54mm_Vertical, symbol Connector_Generic:Conn_01x05
- added R13: 220k, Resistor_THT:R_Axial_DIN0207_L6.3mm_D2.5mm_P2.54mm_Vertical, symbol Device:R_US
- added R14: 47k, Resistor_THT:R_Axial_DIN0207_L6.3mm_D2.5mm_P2.54mm_Vertical, symbol Device:R_US
- added TP10: B2, TestPoint:TestPoint_Loop_D2.54mm_Drill1.5mm_Beaded, symbol Connector:TestPoint
- added TP11: B3, TestPoint:TestPoint_Loop_D2.54mm_Drill1.5mm_Beaded, symbol Connector:TestPoint
- added TP6: Clk, TestPoint:TestPoint_Loop_D2.54mm_Drill1.5mm_Beaded, symbol Connector:TestPoint
- added TP7: DAC, TestPoint:TestPoint_Loop_D2.54mm_Drill1.5mm_Beaded, symbol Connector:TestPoint
- added TP8: B0, TestPoint:TestPoint_Loop_D2.54mm_Drill1.5mm_Beaded, symbol Connector:TestPoint
- added TP9: B1, TestPoint:TestPoint_Loop_D2.54mm_Drill1.5mm_Beaded, symbol Connector:TestPoint
- added U4: NE555P, Package_DIP:DIP-8_W7.62mm, symbol Timer:NE555P
- C1: footprint (none) -> Capacitor_THT:C_Rect_L7.0mm_W3.5mm_P5.00mm
- Q1: now not fitted
- R1, R10, R11, R12, R2, R3, R4, R5, R6, R8, R9: footprint (none) -> Resistor_THT:R_Axial_DIN0207_L6.3mm_D2.5mm_P2.54mm_Vertical
- R7: value 220k -> 100k; footprint (none) -> Resistor_THT:R_Axial_DIN0207_L6.3mm_D2.5mm_P2.54mm_Vertical
- TP1, TP2, TP3, TP4, TP5: footprint (none) -> TestPoint:TestPoint_Loop_D2.54mm_Drill1.5mm_Beaded
- U1: footprint (none) -> Package_DIP:DIP-8_W7.62mm_Socket_LongPads
- U2: footprint (none) -> Package_DIP:DIP-14_W7.62mm_Socket_LongPads
- U3: value ~ -> AD557; footprint (none) -> Package_DIP:DIP-16_W7.62mm_Socket_LongPads; Alternate (none) -> MX7224, AD5330
Connections:
- net +5V: now also R13.1, U4.4 (R), U4.8 (VCC)
- net Clock: now also R14.2, TP6.1, U4.3 (Q)
- net GND: now also U2.12 (MR), C2.2, C3.2, J1.2 (Pin_2), J1.5 (Pin_5), U4.1 (GND)
- net Stair: now also TP7.1
- net C: now reaches Q1.3 (C), Q2.2 (B), Q2.3 (C), Q3.2 (B), TP1.1, TP4.1
- net C: now also J1.1 (Pin_1), J1.4 (Pin_4)
- net at U2.5 (Q2), U3.1 (BIT_8): now also TP10.1
- net at U2.4 (Q1), U3.2 (BIT_7): now also TP9.1
- net at U2.3 (Q0), U3.3 (BIT_6): now also TP8.1
- net B: now reaches Q1.2 (B), R7.2, TP2.1
- net B: now also J1.3 (Pin_3)
- net at U2.6 (Q3): now also TP11.1
- new net: C3.1, U4.5 (CV)
- new net: C2.1, R13.2, R14.1, U4.2 (TR), U4.6 (THR)
- no-connect marks 0 -> 1
Other:
- note added: "DUT"
- note added: "Max 2.53V"
- moved on the sheet: U2C
